File: layouts/default/default.kicad_pcb (KiCad board)
At the start: 2 copper layers, 0 parts

Commit message: example resistor-capacitor connection
Parts:
- added C1: 100nF ±10% 16V X7R, Samsung_Electro_Mechanics_CL05B104KO5NNNC:C0402, F.Cu at (0.00, 0.00)
- added R1: 10kΩ ±1% 62.5mW, UNI_ROYAL_0402WGF1002TCE:R0402, F.Cu at (0.00, -10.0)
